File: SensorFCPlus/Antenna_Diversity/ExpressLRS_2.4GHz/Version_2_M10Q_QMC5883L/Version_2_M10Q_QMC5883L/SE2431L.kicad_sch (KiCad schematic)
At the start: 8 parts, among them U7 SE2431L-R

Commit message: Update README.md and Version 2 files; add new GIF and MP4 for Version 2
Other:
- company: (none) -> https://github.com/Paschalis
- title: (none) -> SE2431L
Changed lines of the file:
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@@
 	(generator_version "8.0")
 	(paper "A4")
+	(title_block
+		(title "SE2431L")
+		(date "2025-01-28")
+		(rev "1.0")
+		(company "https://github.com/Paschalis")
+		(comment 2 "switch with support for antenna diversity.")
+		(comment 3 "Integrates a power amplifier (PA), a low noise amplifier (LNA), and an RF")
+	)
 	(junction
 		(at 151.13 135.89)
@@
 	(label "BOUT"
 		(at 101.6 59.69 180)
-		(fields_autoplaced yes)
 		(effects
 			(font
@@
 	(label "VCC2"
 		(at 130.81 135.89 180)
-		(fields_autoplaced yes)
 		(effects
 			(font
@@
 	(label "BOUT"
 		(at 168.91 63.5 0)
-		(fields_autoplaced yes)
 		(effects
 			(font
@@
 	(label "VCC1"
 		(at 130.81 111.76 180)
-		(fields_autoplaced yes)
 		(effects
 			(font
@@
 	(label "VCC2"
 		(at 168.91 73.66 0)
-		(fields_autoplaced yes)
 		(effects
 			(font
@@
 	(label "VCC1"
 		(at 168.91 66.04 0)
-		(fields_autoplaced yes)
 		(effects
 			(font
@@
 		(shape input)
 		(at 177.8 60.96 0)
-		(fields_autoplaced yes)
 		(effects
 			(font
@@
 		(shape output)
 		(at 172.72 88.9 0)
-		(fields_autoplaced yes)
 		(effects
 			(font
@@
 		(shape output)
 		(at 172.72 83.82 0)
-		(fields_autoplaced yes)
 		(effects
 			(font
@@
 		(shape input)
 		(at 172.72 81.28 0)
-		(fields_autoplaced yes)
 		(effects
 			(font
@@
 		(shape input)
 		(at 115.57 71.12 180)
-		(fields_autoplaced yes)
-		(effects
-			(font
+		(effects
+			(font
