File: SensorFCPlus/Antenna_Diversity/ExpressLRS_2.4GHz/Version_2_M10Q_QMC5883L/Version_2_M10Q_QMC5883L/SX1280.kicad_sch (KiCad schematic)
At the start: 8 parts, among them U6 SX1280IMLTRT, Y2 52MHz

Commit message: Update README.md and Version 2 files; add new GIF and MP4 for Version 2
Other:
- company: (none) -> https://github.com/Paschalis
- title: (none) -> SX1280
Changed lines of the file:
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@@
 	(generator_version "8.0")
 	(paper "A4")
+	(title_block
+		(title "SX1280")
+		(date "2025-01-28")
+		(rev "1.0")
+		(company "https://github.com/Paschalis")
+		(comment 2 "capabilities in LoRa communication, making it ideal for reliable telemetry.")
+		(comment 3 "The SX1280 is used for its long-range, low-power, and high-performance ")
+	)
 	(junction
 		(at 129.54 60.96)
@@
 	(label "VDD_INN"
 		(at 58.42 86.36 180)
-		(fields_autoplaced yes)
 		(effects
 			(font
@@
 	(label "RFIO"
 		(at 129.54 66.04 0)
-		(fields_autoplaced yes)
 		(effects
 			(font
@@
 	(label "VDD_INN"
 		(at 67.31 60.96 180)
-		(fields_autoplaced yes)
 		(effects
 			(font
@@
 	(label "RFIO"
 		(at 209.55 77.47 180)
-		(fields_autoplaced yes)
 		(effects
 			(font
@@
 		(shape input)
 		(at 129.54 76.2 0)
-		(fields_autoplaced yes)
 		(effects
 			(font
@@
 		(shape bidirectional)
 		(at 67.31 76.2 180)
-		(fields_autoplaced yes)
 		(effects
 			(font
@@
 		(shape input)
 		(at 129.54 73.66 0)
-		(fields_autoplaced yes)
 		(effects
 			(font
@@
 		(shape output)
 		(at 129.54 81.28 0)
-		(fields_autoplaced yes)
 		(effects
 			(font
@@
 		(shape output)
 		(at 67.31 73.66 180)
-		(fields_autoplaced yes)
 		(effects
 			(font
@@
 		(shape input)
 		(at 67.31 63.5 180)
-		(fields_autoplaced yes)
 		(effects
 			(font
@@
 		(shape output)
 		(at 245.11 77.47 0)
-		(fields_autoplaced yes)
 		(effects
 			(font
@@
 		(shape input)
 		(at 129.54 78.74 0)
-		(fields_autoplaced yes)
-		(effects
-			(font
+		(effects
+			(font
