File: SensorFCPlus/Antenna_Diversity/ExpressLRS_2.4GHz/Version_1_M10Q_HMC5883L/Version_1_M10Q_HMC5883L/SX1280.kicad_sch (KiCad schematic)
At the start: 8 parts, among them U6 SX1280IMLTRT, Y2 52MHz

Commit message: Updated README and V1 M10Q HMC5883L KiCad files, added documentation and media
Other:
- title: (none) -> SX1280
