File: SensorFCPlus/Antenna_Diversity/ExpressLRS_2.4GHz/Version_3_M10Q_LSM303AH/Version_3_M10Q_LSM303AH/SX1280.kicad_sch (KiCad schematic)
At the start: 8 parts, among them U6 SX1280IMLTRT, Y2 52MHz

Commit message: Update PCB design for Version 3 M10Q LSM303AH (ESP8285, SE2431L, SX1280, and main board)
Parts:
- C24, C25, C26, C27, C28: footprint Capacitor_SMD:C_0805_2012Metric_Pad1.18x1.45mm_HandSolder -> Capacitor_SMD:C_0603_1608Metric_Pad1.08x0.95mm_HandSolder
Changed lines of the file:
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@@
 			)
 		)
-		(property "Footprint" "Capacitor_SMD:C_0805_2012Metric_Pad1.18x1.45mm_HandSolder"
+		(property "Footprint" "Capacitor_SMD:C_0603_1608Metric_Pad1.08x0.95mm_HandSolder"
 			(at 71.12 92.71 0)
 			(effects
@@
 			)
 		)
-		(property "Footprint" "Capacitor_SMD:C_0805_2012Metric_Pad1.18x1.45mm_HandSolder"
+		(property "Footprint" "Capacitor_SMD:C_0603_1608Metric_Pad1.08x0.95mm_HandSolder"
 			(at 48.26 92.71 0)
 			(effects
@@
 			)
 		)
-		(property "Footprint" "Capacitor_SMD:C_0805_2012Metric_Pad1.18x1.45mm_HandSolder"
+		(property "Footprint" "Capacitor_SMD:C_0603_1608Metric_Pad1.08x0.95mm_HandSolder"
 			(at 57.15 59.69 0)
 			(effects
@@
 			)
 		)
-		(property "Footprint" "Capacitor_SMD:C_0805_2012Metric_Pad1.18x1.45mm_HandSolder"
+		(property "Footprint" "Capacitor_SMD:C_0603_1608Metric_Pad1.08x0.95mm_HandSolder"
 			(at 146.05 88.9 0)
 			(effects
@@
 			)
 		)
-		(property "Footprint" "Capacitor_SMD:C_0805_2012Metric_Pad1.18x1.45mm_HandSolder"
+		(property "Footprint" "Capacitor_SMD:C_0603_1608Metric_Pad1.08x0.95mm_HandSolder"
 			(at 62.23 92.71 0)
 			(effects

Commit message: Updated Version_3_M10Q_LSM303AH
Other:
- title: (none) -> SX1280
Changed lines of the file:
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@@
 	(paper "A4")
 	(title_block
+		(title "SX1280")
 		(date "05-01-2025")
 		(rev "1.0")
@@
 	(label "VDD_INN"
 		(at 59.69 87.63 180)
-		(fields_autoplaced yes)
 		(effects
 			(font
@@
 	(label "VDD_INN"
 		(at 68.58 62.23 180)
-		(fields_autoplaced yes)
 		(effects
 			(font
@@
 	(label "RFIO"
 		(at 210.82 78.74 180)
-		(fields_autoplaced yes)
 		(effects
 			(font
@@
 	(label "RFIO"
 		(at 130.81 67.31 0)
-		(fields_autoplaced yes)
 		(effects
 			(font
@@
 		(shape input)
 		(at 130.81 77.47 0)
-		(fields_autoplaced yes)
 		(effects
 			(font
@@
 		(shape bidirectional)
 		(at 68.58 77.47 180)
-		(fields_autoplaced yes)
 		(effects
 			(font
@@
 		(shape input)
 		(at 68.58 64.77 180)
-		(fields_autoplaced yes)
 		(effects
 			(font
@@
 		(shape output)
 		(at 130.81 82.55 0)
-		(fields_autoplaced yes)
 		(effects
 			(font
@@
 		(shape input)
 		(at 130.81 74.93 0)
-		(fields_autoplaced yes)
 		(effects
 			(font
@@
 		(shape output)
 		(at 68.58 74.93 180)
-		(fields_autoplaced yes)
 		(effects
 			(font
@@
 		(shape input)
 		(at 130.81 80.01 0)
-		(fields_autoplaced yes)
 		(effects
 			(font
@@
 		(shape output)
 		(at 246.38 78.74 0)
-		(fields_autoplaced yes)
-		(effects
-			(font
+		(effects
+			(font
